File: MCU Datalogger.kicad_sch (KiCad schematic)
At the start: 0 parts

Commit message: Setup of EEschema for new project.
Other:
- title: (none) -> ${project_name}
Changed lines of the file:
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@@
 (kicad_sch (version 20210621) (generator eeschema)
   (paper "A4")
-  (symbol_instances)
+  (title_block
+    (title "${project_name}")
+    (date "2021-07-21")
+    (rev "1")
+  )
+  (sheet_instances
+    (path "/" (page "1"))
+  )
 )
