File: MCU Datalogger.kicad_sch (KiCad schematic)
At the start: 25 parts, among them U1 24LC1025, U2 DS1337S+, U3 24LC1025, U4 ATMEGA328P-AU, Y1 32.768 KHz, Y2 16 MHz

Commit message: Generated BOM.
Parts:
- U2: Purpose (none) -> Test string in purpose field; Wikipedia URL (none) -> https://en.wikipedia.org/wiki/Real-time_clock
Changed lines of the file:
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@@
       (effects (font (size 1.27 1.27)) (justify left bottom) hide)
+    )
+    (property "Purpose" "Test string in purpose field" (id 4) (at 67.31 62.23 0)
+      (effects (font (size 1.27 1.27)) hide)
+    )
+    (property "Wikipedia URL" "https://en.wikipedia.org/wiki/Real-time_clock" (id 5) (at 67.31 62.23 0)
+      (effects (font (size 1.27 1.27)) hide)
     )
     (pin "1")
