File: MCU Datalogger.kicad_pcb (KiCad board)
At the start: 0 parts

Commit message: Fixing typos.
Parts:
- added BT1: Battery, Connector_PinHeader_2.54mm:PinHeader_1x02_P2.54mm_Vertical, F.Cu at (209.0, 89.4)
- added C1: 0.1uF, Capacitor_SMD:C_0805_2012Metric, F.Cu at (202.5, 98.9)
- added C2: 22pF, Capacitor_SMD:C_0805_2012Metric, F.Cu at (207.0, 101.5)
- added C3: 22pF, Capacitor_SMD:C_0805_2012Metric, F.Cu at (203.0, 88.8)
- added C4: 0.1uF, Capacitor_SMD:C_0805_2012Metric, F.Cu at (219.3, 87.8)
- added C5: 100nF, Capacitor_SMD:C_0805_2012Metric, F.Cu at (202.5, 101.9)
- added D1: LED, LED_SMD:LED_0805_2012Metric, F.Cu at (198.6, 88.8)
- added D2: LED, LED_SMD:LED_0805_2012Metric, F.Cu at (224.1, 82.1)
- added H1: MountingHole, MountingHole:MountingHole_2.1mm, F.Cu at (207.8, 97.2)
- added H2: MountingHole, MountingHole:MountingHole_2.1mm, F.Cu at (197.4, 102.2)
- added H3: MountingHole, MountingHole:MountingHole_2.1mm, F.Cu at (219.0, 83.4)
- added H4: MountingHole, MountingHole:MountingHole_2.1mm, F.Cu at (214.2, 90.0)
- added J1: Conn_01x04_Male, Connector_PinHeader_2.54mm:PinHeader_1x04_P2.54mm_Vertical, F.Cu at (244.1, 82.9)
- added J2: Conn_01x09_Male, Connector_PinHeader_2.54mm:PinHeader_1x09_P2.54mm_Vertical, F.Cu at (234.8, 82.9)
- added J3: Conn_01x04_Male, Connector_PinHeader_2.54mm:PinHeader_1x04_P2.54mm_Vertical, F.Cu at (239.5, 82.9)
- added J4: Conn_02x03_Odd_Even, Connector_PinHeader_2.54mm:PinHeader_2x03_P2.54mm_Vertical, F.Cu at (248.8, 82.9)
- added R1: 10K, Resistor_SMD:R_0805_2012Metric, F.Cu at (212.9, 97.3)
- added R2: 10K, Resistor_SMD:R_0805_2012Metric, F.Cu at (211.4, 101.5)
- added R3: 4.7K, Resistor_SMD:R_0805_2012Metric, F.Cu at (224.1, 85.0)
- added R4: 4.7K, Resistor_SMD:R_0805_2012Metric, F.Cu at (223.8, 88.0)
- added R5: 330, Resistor_SMD:R_0805_2012Metric, F.Cu at (218.0, 94.3)
- added R6: 10K, Resistor_SMD:R_0805_2012Metric, F.Cu at (219.3, 90.8)
- added R7: 330, Resistor_SMD:R_0805_2012Metric, F.Cu at (213.6, 94.3)
- added U1: 24LC1025, Package_SO:SOIC-8_5.23x5.23mm_P1.27mm, F.Cu at (201.5, 83.9)
- added U2: DS1337S+, Footprints:SOIC127P600X175-8N, F.Cu at (211.9, 83.8)
- added U3: 24LC1025, Package_SO:SOIC-8_5.23x5.23mm_P1.27mm, F.Cu at (189.5, 96.0)
- added U4: ATMEGA328P-AU, Footprints:QFP80P900X900X120-32N, F.Cu at (190.3, 86.6)
- added Y1: 32.768 KHz, Crystal:Crystal_SMD_5032-2Pin_5.0x3.2mm_HandSoldering, F.Cu at (189.4, 101.8)
- added Y2: 16 MHz, Crystal:Crystal_SMD_5032-2Pin_5.0x3.2mm_HandSoldering, F.Cu at (199.8, 95.0)
Other:
- copper layers 0 -> 2
